File: monKWH-prototype(110x75)/untitled.sch (EAGLE design)
At the start: 25 parts, among them X1 MSTBA2

Commit message: menambahkan komponen coaxial conn
Parts:
- added J1: U.FL-R-SMT(01), U.FL-R-SMT_01_:U.FL-R-SMT(01)
Connections:
- new net ANT: J1.SIG, LORA-NICERF-V1.ANT
- net GND: now also J1.GND
Changed lines of the file:
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@@
 <part name="SV1" library="con-lstb" library_urn="urn:adsk.eagle:library:162" deviceset="MA04-1" device="" package3d_urn="urn:adsk.eagle:package:8337/1"/>
 <part name="GND3" library="supply1" library_urn="urn:adsk.eagle:library:371" deviceset="GND" device=""/>
+<part name="J1" library="U.FL-R-SMT_01_" deviceset="U.FL-R-SMT(01)" device=""/>
 </parts>
 <sheets>
@@
 <attribute name="VALUE" x="68.58" y="30.48" size="1.778" layer="96"/>
 </instance>
+<instance part="J1" gate="G$1" x="17.78" y="-30.48" smashed="yes">
+<attribute name="NAME" x="13.96143125" y="-26.40686875" size="1.27285" layer="95"/>
+<attribute name="VALUE" x="13.45218125" y="-36.0807" size="1.27288125" layer="96"/>
+</instance>
 </instances>
 <busses>
@@
 <wire x1="35.56" y1="-27.94" x2="35.56" y2="-25.4" width="0.1524" layer="91"/>
 <junction x="35.56" y="-25.4"/>
+<pinref part="J1" gate="G$1" pin="GND"/>
+<wire x1="7.62" y1="-33.02" x2="35.56" y2="-33.02" width="0.1524" layer="91"/>
+<wire x1="35.56" y1="-33.02" x2="35.56" y2="-27.94" width="0.1524" layer="91"/>
+<junction x="35.56" y="-27.94"/>
 </segment>
 <segment>
@@
 </segment>
 </net>
+<net name="ANT" class="0">
+<segment>
+<pinref part="LORA-NICERF-V1" gate="G$1" pin="ANT"/>
+<wire x1="22.86" y1="-7.62" x2="25.4" y2="-7.62" width="0.1524" layer="91"/>
+<label x="25.4" y="-7.62" size="1.778" layer="95" xref="yes"/>
+</segment>
+<segment>
+<pinref part="J1" gate="G$1" pin="SIG"/>
+<wire x1="7.62" y1="-27.94" x2="5.08" y2="-27.94" width="0.1524" layer="91"/>
+<label x="5.08" y="-27.94" size="1.778" layer="95" rot="R180" xref="yes"/>
+</segment>
+</net>
