File: monKWH-prototype(110x75)/untitled.sch (EAGLE design)
At the start: 26 parts, among them J1 U.FL-R-SMT(01), X1 MSTBA2

Commit message: revisi .brd
Parts:
- removed JP3: (no value), pinhead:PINHD-1X2
- added JP4: (no value), pinhead:PINHD-1X3
Connections:
- net N$5: now also JP4.3; no longer JP3.2
- net N$8: now also JP4.1; no longer JP3.1
Changed lines of the file:
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@@
 <part name="JP2" library="pinhead" library_urn="urn:adsk.eagle:library:325" deviceset="PINHD-1X2" device="" package3d_urn="urn:adsk.eagle:package:22435/2"/>
 <part name="X1" library="con-phoenix-508" library_urn="urn:adsk.eagle:library:176" deviceset="MSTBA2" device="" package3d_urn="urn:adsk.eagle:package:9615/1"/>
-<part name="JP3" library="pinhead" library_urn="urn:adsk.eagle:library:325" deviceset="PINHD-1X2" device="" package3d_urn="urn:adsk.eagle:package:22435/2"/>
 <part name="POWER" library="led" library_urn="urn:adsk.eagle:library:259" deviceset="TLLR4400" device="" package3d_urn="urn:adsk.eagle:package:15797/1"/>
 <part name="PROSES" library="led" library_urn="urn:adsk.eagle:library:259" deviceset="TLLR4400" device="" package3d_urn="urn:adsk.eagle:package:15797/1"/>
@@
 <part name="GND3" library="supply1" library_urn="urn:adsk.eagle:library:371" deviceset="GND" device=""/>
 <part name="J1" library="U.FL-R-SMT_01_" deviceset="U.FL-R-SMT(01)" device=""/>
+<part name="JP4" library="pinhead" library_urn="urn:adsk.eagle:library:325" deviceset="PINHD-1X3" device="" package3d_urn="urn:adsk.eagle:package:22458/2"/>
 </parts>
 <sheets>
@@
 <attribute name="NAME" x="72.009" y="171.704" size="1.778" layer="95" rot="R90"/>
 </instance>
-<instance part="JP3" gate="G$1" x="73.66" y="144.78" smashed="yes" rot="R270">
-<attribute name="NAME" x="79.375" y="151.13" size="1.778" layer="95" rot="R270"/>
-<attribute name="VALUE" x="68.58" y="151.13" size="1.778" layer="96" rot="R270"/>
-</instance>
 <instance part="POWER" gate="G$1" x="-76.2" y="-106.68" smashed="yes">
 <attribute name="NAME" x="-72.644" y="-111.252" size="1.778" layer="95" rot="R90"/>
@@
 <attribute name="NAME" x="13.96143125" y="-26.40686875" size="1.27285" layer="95"/>
 <attribute name="VALUE" x="13.45218125" y="-36.0807" size="1.27288125" layer="96"/>
+</instance>
+<instance part="JP4" gate="A" x="73.66" y="142.24" smashed="yes" rot="R270">
+<attribute name="NAME" x="79.375" y="148.59" size="1.778" layer="95" rot="R270"/>
+<attribute name="VALUE" x="66.04" y="148.59" size="1.778" layer="96" rot="R270"/>
 </instance>
 </instances>
@@
 <net name="N$5" class="0">
 <segment>
-<pinref part="JP3" gate="G$1" pin="2"/>
 <pinref part="X1" gate="-2" pin="1"/>
-<wire x1="73.66" y1="147.32" x2="71.12" y2="147.32" width="0.1524" layer="91"/>
-<wire x1="71.12" y1="147.32" x2="71.12" y2="160.02" width="0.1524" layer="91"/>
+<wire x1="71.12" y1="144.78" x2="71.12" y2="160.02" width="0.1524" layer="91"/>
+<pinref part="JP4" gate="A" pin="3"/>
 </segment>
 </net>
@@
 <segment>
 <pinref part="X1" gate="-1" pin="1"/>
-<pinref part="JP3" gate="G$1" pin="1"/>
-<wire x1="76.2" y1="160.02" x2="76.2" y2="147.32" width="0.1524" layer="91"/>
-</segment>
-</net>
+<wire x1="76.2" y1="160.02" x2="76.2" y2="144.78" width="0.1524" layer="91"/>
+<pinref part="JP4" gate="A" pin="1"/>
+</segment>
+</net>

Commit message: perubahan mikro dan penambahan Jack-DC
Parts:
- removed U$6: ESP32DEVKITC, ESP32-DEVKITC:ESP32DEVKITC
- added J2: DCJ0202, con-jack:DCJ0202
- added U1: ESP32-DEVKITC-32D, ESP32-DEVKITC-32D:ESP32-DEVKITC-32D
- R2: device adafruit:R-US_M0805 -> 1N5819HW-7:1N5819HW-7
Connections:
- removed net EN: U$6.EN
- removed net RST_LAN1: U$6.IO33
- net 3V3: now also U1.3V3; no longer U$6.3V3
- net GND: now also J2.2, J2.3, U1.GND1, U1.GND2, U1.GND3; no longer U$6.GND@14, U$6.GND@32, U$6.GND@38
- net LED_PROSES: now also U1.IO27; no longer U$6.IO27
- net LED_WARNING: now also U1.IO15; no longer U$6.IO15
- net LORA_DI0: now also U1.IO25; no longer U$6.IO25
- net LORA_DI1: now also U1.IO32; no longer U$6.IO32
- net MISO_HSPI: now also U1.IO12; no longer U$6.IO12
- net MISO_VSPI: now also U1.IO23; no longer U$6.IO23
- net MOSI_HSPI: now also U1.IO13; no longer U$6.IO13
- net MOSI_VSPI: now also U1.IO19; no longer U$6.IO19
- net N$4: now also J2.1
- net N$7: now also R2.A; no longer R2.2
- net OUT+: now also R2.K, U1.EXT_5V; no longer R2.1, U$6.5V
- net RST: now also U1.IO0; no longer U$6.IO0
- net RST_LORA: now also U1.IO26; no longer U$6.IO26
- net RX_DB9: now also U1.IO16; no longer U$6.IO16
- net SCK_HSPI: now also U1.IO14; no longer U$6.IO14
- net SCK_VSPI: now also U1.IO18; no longer U$6.IO18
- net SCL: now also U1.IO22; no longer U$6.IO22
- net SDA: now also U1.IO21; no longer U$6.IO21
- net SS_LAN_CONV: now also U1.IO4; no longer U$6.IO4
- net SS_LORA: now also U1.IO5; no longer U$6.IO5
- net TX_DB9: now also U1.IO17; no longer U$6.IO17
