File: monKWH-prototype(110x75)/untitled.brd (EAGLE design)
At the start: 69 x 109 mm, 26 parts, among them J1 U.FL-R-SMT(01), X1 MSTBA2

Commit message: revisi dimensi
Routing:
- net RX_DB9: track 233.6 -> 230.8 mm
- net GND: track 425.8 -> 423.1 mm
- net MISO_HSPI: track 89.3 -> 88.2 mm
Other:
- board size 69 x 109 mm -> 69.4 x 109.6 mm
Changed lines of the file:
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@@
 <setting verticaltext="up"/>
 </settings>
-<grid distance="0.003125" unitdist="mic" unit="mm" style="lines" multiple="1" display="yes" altdistance="5" altunitdist="mil" altunit="mil"/>
+<grid distance="0.1" unitdist="mm" unit="mm" style="lines" multiple="1" display="yes" altdistance="5" altunitdist="mil" altunit="mil"/>
 <layers>
 <layer number="1" name="Top" color="4" fill="1" visible="yes" active="yes"/>
@@
 <board>
 <plain>
-<wire x1="-3" y1="-1" x2="66" y2="-1" width="0" layer="20"/>
-<wire x1="66" y1="-1" x2="66" y2="108" width="0" layer="20"/>
-<wire x1="66" y1="108" x2="-3" y2="108" width="0" layer="20"/>
-<wire x1="-3" y1="108" x2="-3" y2="-1" width="0" layer="20"/>
-<dimension x1="-3" y1="-1" x2="-3" y2="108" x3="-8" y3="53.5" textsize="1.778" layer="21"/>
-<dimension x1="-3" y1="108" x2="66" y2="108" x3="31.5" y3="119" textsize="1.778" layer="21"/>
+<wire x1="-3.2" y1="-1.3" x2="66.2" y2="-1.3" width="0" layer="20"/>
+<wire x1="66.2" y1="-1.3" x2="66.2" y2="108.3" width="0" layer="20"/>
+<wire x1="66.2" y1="108.3" x2="-3.2" y2="108.3" width="0" layer="20"/>
+<wire x1="-3.2" y1="108.3" x2="-3.2" y2="-1.3" width="0" layer="20"/>
 <dimension x1="66" y1="108" x2="45" y2="108" x3="55.5" y3="113" textsize="1.778" layer="21"/>
 <dimension x1="33" y1="108" x2="45" y2="108" x3="39" y3="113" textsize="1.778" layer="21"/>
 <dimension x1="51" y1="107" x2="54" y2="107" x3="52.5" y3="110" textsize="1.778" layer="21"/>
 <dimension x1="66" y1="-1" x2="56" y2="-1" x3="61" y3="-5" textsize="1.778" layer="21"/>
+<dimension x1="-3.2" y1="108.3" x2="-3.2" y2="-1.3" x3="-12.3" y3="53.5" textsize="1.778" layer="21"/>
+<dimension x1="-3.2" y1="108.3" x2="66.2" y2="108.3" x3="31.5" y3="126" textsize="1.778" layer="21"/>
 </plain>
 <attributes>
@@
 <wire x1="47.74153125" y1="88.867828125" x2="47.3627625" y2="88.867828125" width="0.4064" layer="1"/>
 <wire x1="46.521059375" y1="88.867828125" x2="45.46480625" y2="88.867828125" width="0.4064" layer="1"/>
-<wire x1="45.46480625" y1="88.867828125" x2="38.284215625" y2="88.867828125" width="0.4064" layer="1"/>
-<wire x1="34.7496" y1="92.40244375" x2="32.923290625" y2="92.40244375" width="0.4064" layer="1"/>
+<wire x1="45.46480625" y1="88.867828125" x2="36.45790625" y2="88.867828125" width="0.4064" layer="1"/>
+<wire x1="36.45790625" y1="88.867828125" x2="32.923290625" y2="92.40244375" width="0.4064" layer="1"/>
 <via x="32.923290625" y="92.40244375" extent="1-16" drill="1"/>
 <wire x1="32.923290625" y1="92.40244375" x2="28.736528125" y2="92.40244375" width="0.4064" layer="16"/>
 <wire x1="28.736528125" y1="92.40244375" x2="27.663496875" y2="91.3294125" width="0.4064" layer="16"/>
-<wire x1="38.284215625" y1="88.867828125" x2="34.7496" y2="92.40244375" width="0.4064" layer="1"/>
 <wire x1="54.7300125" y1="104.31539375" x2="52.97211875" y2="102.5575" width="0.4064" layer="16"/>
 <wire x1="7" y1="31.73" x2="5.83983125" y2="31.73" width="0.4064" layer="16"/>
@@
 <via x="53.7688375" y="9.062490625" extent="1-16" drill="1"/>
 <wire x1="53.7688375" y1="9.062490625" x2="51.59269375" y2="11.238634375" width="0.4064" layer="1"/>
-<wire x1="51.59269375" y1="40.371728125" x2="48.419153125" y2="43.54526875" width="0.4064" layer="1"/>
-<wire x1="48.419153125" y1="43.54526875" x2="48.419153125" y2="47.121590625" width="0.4064" layer="1"/>
+<wire x1="51.59269375" y1="11.238634375" x2="51.59269375" y2="50.29513125" width="0.4064" layer="1"/>
 <wire x1="55.23578125" y1="53.93821875" x2="55.23578125" y2="61.10209375" width="0.4064" layer="1"/>
 <via x="55.23578125" y="61.10209375" extent="1-16" drill="1"/>
 <wire x1="55.026525" y1="61.31135" x2="55.026525" y2="61.79241875" width="0.4064" layer="16"/>
 <wire x1="55.026525" y1="61.79241875" x2="55.026525" y2="62.471025" width="0.4064" layer="16"/>
-<wire x1="51.59269375" y1="11.238634375" x2="51.59269375" y2="40.371728125" width="0.4064" layer="1"/>
-<wire x1="48.419153125" y1="47.121590625" x2="55.23578125" y2="53.93821875" width="0.4064" layer="1"/>
+<wire x1="51.59269375" y1="50.29513125" x2="55.23578125" y2="53.93821875" width="0.4064" layer="1"/>
 <contactref element="J1" pad="2"/>
 <contactref element="J1" pad="1"/>
@@
 <via x="46.317503125" y="33.755259375" extent="1-16" drill="1"/>
 <wire x1="46.317503125" y1="33.755259375" x2="46.317503125" y2="36.237809375" width="0.4064" layer="1"/>
-<via x="32.70110625" y="89.96884375" extent="1-16" drill="1"/>
-<wire x1="32.70110625" y1="89.96884375" x2="31.521675" y2="88.7894125" width="0.4064" layer="16"/>
-<wire x1="31.521675" y1="88.7894125" x2="27.663496875" y2="88.7894125" width="0.4064" layer="16"/>
+<via x="32.43305625" y="89.4864875" extent="1-16" drill="1"/>
+<wire x1="32.43305625" y1="89.4864875" x2="31.73598125" y2="88.7894125" width="0.4064" layer="16"/>
+<wire x1="31.73598125" y1="88.7894125" x2="27.663496875" y2="88.7894125" width="0.4064" layer="16"/>
 <wire x1="37.607003125" y1="20.685921875" x2="37.607003125" y2="23.886503125" width="0.4064" layer="16"/>
 <wire x1="37.607003125" y1="23.886503125" x2="42.006159375" y2="28.285659375" width="0.4064" layer="16"/>
@@
 <wire x1="40.0442125" y1="50.555096875" x2="34.8249125" y2="50.555096875" width="0.4064" layer="1"/>
 <wire x1="34.8249125" y1="50.555096875" x2="32.3644375" y2="53.015571875" width="0.4064" layer="1"/>
-<wire x1="32.3644375" y1="53.015571875" x2="32.3644375" y2="89.632175" width="0.4064" layer="1"/>
-<wire x1="32.3644375" y1="89.632175" x2="32.70110625" y2="89.96884375" width="0.4064" layer="1"/>
+<wire x1="32.3644375" y1="53.015571875" x2="32.3644375" y2="89.41786875" width="0.4064" layer="1"/>
+<wire x1="32.3644375" y1="89.41786875" x2="32.43305625" y2="89.4864875" width="0.4064" layer="1"/>
 <wire x1="42.575309375" y1="39.980003125" x2="42.575309375" y2="48.024" width="0.4064" layer="1"/>
 </signal>
@@
 <wire x1="18.373196875" y1="26.761553125" x2="18.52289375" y2="26.91125" width="0.4064" layer="16"/>
 <wire x1="53.59765625" y1="73.550371875" x2="53.59765625" y2="53.909353125" width="0.4064" layer="1"/>
-<wire x1="53.59765625" y1="53.909353125" x2="47.004034375" y2="47.31573125" width="0.4064" layer="1"/>
-<wire x1="47.004034375" y1="42.580240625" x2="50.478096875" y2="39.106178125" width="0.4064" layer="1"/>
-<wire x1="50.478096875" y1="39.106178125" x2="50.478096875" y2="13.819134375" width="0.4064" layer="1"/>
+<wire x1="53.59765625" y1="53.909353125" x2="50.478096875" y2="50.78979375" width="0.4064" layer="1"/>
 <wire x1="50.478096875" y1="13.819134375" x2="40.575978125" y2="3.917015625" width="0.4064" layer="1"/>
 <wire x1="59.711640625" y1="79.66435625" x2="53.59765625" y2="73.550371875" width="0.4064" layer="1"/>
-<wire x1="47.004034375" y1="47.31573125" x2="47.004034375" y2="42.580240625" width="0.4064" layer="1"/>
+<wire x1="50.478096875" y1="50.78979375" x2="50.478096875" y2="13.819134375" width="0.4064" layer="1"/>
 </signal>
 <signal name="MISO_VSPI">
@@
 <signal name="N$2">
 <polygon width="0.4064" layer="16" isolate="1.016">
-<vertex x="-3" y="108"/>
-<vertex x="66" y="108"/>
-<vertex x="66" y="-1"/>
-<vertex x="-3" y="-1"/>
+<vertex x="-3.2" y="108.3"/>
+<vertex x="66.2" y="108.3"/>
+<vertex x="66.2" y="-1.3"/>
+<vertex x="-3.2" y="-1.3"/>
 </polygon>
 </signal>
 <signal name="N$9">
 <polygon width="0.4064" layer="1" isolate="1.016">
-<vertex x="-3" y="108"/>
-<vertex x="66" y="108"/>
-<vertex x="66" y="-1"/>
-<vertex x="-3" y="-1"/>
+<vertex x="-3.2" y="108.3"/>
+<vertex x="66.2" y="108.3"/>
+<vertex x="66.2" y="-1.3"/>
+<vertex x="-3.2" y="-1.3"/>
 </polygon>
 </signal>

Commit message: perubahan mikro dan penambahan Jack-DC
Parts:
- removed U$6: ESP32DEVKITC, ESP32-DEVKITC:ESP32-DEVKITC
- added J2: DCJ0202, con-jack:DCJ0202
- added U1: ESP32-DEVKITC-32D, ESP32-DEVKITC-32D:MODULE_ESP32-DEVKITC-32D
- R2: device adafruit:M0805 -> 1N5819HW-7:SOD3715X145N
- moved S1 110.5 mm to (3.73, 3.93), turned to 0 degrees
- moved C3 97.0 mm to (3.77, 8.15), turned to 0 degrees
- moved J1 6.19 mm to (13.2, 46.7), turned to 180 degrees
- moved U$5 5.06 mm to (39.7, 27.5)
- moved C1 4.69 mm to (48.2, 92.7), turned to 0 degrees
- moved U$3 4.59 mm to (63.5, -0.61)
- moved R1 3.19 mm to (11.1, 32.1)
- moved POWER 2.00 mm to (7.00, 31.0)
- moved PROSES 2.00 mm to (7.00, 41.0)
- moved WARNING 2.00 mm to (7.00, 51.0)
- moved R16 1.41 mm to (10.5, 51.8)
- moved R3 1.25 mm to (10.8, 43.2)
- moved X1 1.19 mm to (39.0, 106.2)
Connections:
- removed net EN: U$6.2
- removed net RST_LAN1: U$6.8
- net 3V3: now also U1.1; no longer U$6.1
- net GND: now also J2.2, J2.3, U1.14, U1.20, U1.26; no longer U$6.14, U$6.32, U$6.38
- net LED_PROSES: now also U1.11; no longer U$6.11
- net LED_WARNING: now also U1.35; no longer U$6.23
- net LORA_DI0: now also U1.9; no longer U$6.9
- net LORA_DI1: now also U1.7; no longer U$6.7
- net MISO_HSPI: now also U1.13; no longer U$6.13
- net MISO_VSPI: now also U1.21; no longer U$6.37
- net MOSI_HSPI: now also U1.15; no longer U$6.15
- net MOSI_VSPI: now also U1.27; no longer U$6.31
- net N$4: now also J2.1
- net N$7: now also R2.A; no longer R2.2
- net OUT+: now also R2.C, U1.19; no longer R2.1, U$6.19
- net RST: now also U1.33; no longer U$6.25
- net RST_LORA: now also U1.10; no longer U$6.10
- net RX_DB9: now also U1.31; no longer U$6.27
- net SCK_HSPI: now also U1.12; no longer U$6.12
- net SCK_VSPI: now also U1.28; no longer U$6.30
- net SCL: now also U1.22; no longer U$6.36
- net SDA: now also U1.25; no longer U$6.33
- net SS_LAN_CONV: now also U1.32; no longer U$6.26
- net SS_LORA: now also U1.29; no longer U$6.29
- net TX_DB9: now also U1.30; no longer U$6.28
Routing:
- net RX_DB9: track 230.8 -> 94.7 mm
- net RST: track 156.7 -> 213.2 mm, vias 0 -> 2
- net N$4: track 23.3 -> 43.9 mm
- net 3V3: track 203.9 -> 217.2 mm
- net TX_DB9: track 77.2 -> 89.2 mm
- net MISO_HSPI: track 88.2 -> 95.9 mm
- net GND: track 423.1 -> 415.7 mm, vias 5 -> 7
- net SS_LAN_CONV: track 108.9 -> 115.5 mm
- net MOSI_HSPI: track 104.9 -> 111.1 mm
- net N$7: track 19.5 -> 24.2 mm, vias 0 -> 1
- net LED_WARNING: track 54.5 -> 58.5 mm
- net SCK_HSPI: track 94.4 -> 98.3 mm
- net OUT+: track 226.0 -> 229.5 mm, vias 3 -> 4
- net ANT: track 6.39 -> 9.29 mm
- net SDA: track 96.3 -> 98.9 mm
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
Commit message: revisi jaulur .brd
Parts:
- moved POWER 1.00 mm to (7.00, 30.0)
- moved PROSES 1.00 mm to (7.00, 40.0)
- moved WARNING 1.00 mm to (7.00, 50.0)
- moved S1 0.17 mm to (3.77, 4.10)
Routing:
- net GND: track 415.7 -> 419.0 mm
- net MOSI_HSPI: track 111.1 -> 110.0 mm
- net N$3: track 5.18 -> 6.18 mm
- net N$8: track 7.72 -> 7.09 mm
- net RST: track 213.2 -> 212.7 mm
- net 3V3: track 217.2 -> 216.7 mm
